File: schematics/Orion68/orion68_serial.kicad_sch (KiCad schematic)
At the start: 65 parts, among them J11 IDE-40W, J12 PWR, J700 Euro96pin, J701 RS232_1, J702 RS232_1, J703 RS232_1, U17 74LS139, U18_C? 100nf, U19 74LS139, U20 74HC138, U701 UART1, U702 UART2, U703 UART3, Y1 14.745600

Commit message: 2026-09-27: implemented and tested Orionide board
Connections:
- net A11: now also U28.5 (I4); no longer U20.4 (~{E0})
- net /AS: now also U20.4 (~{E0}); no longer U28.5 (I4)
Other:
- note added: "FF4000 - FF40FF UART0 FF4100 - FF41FF UART1 FF4200 - FF42FF UART2 FF4300 - FF43FF UART3 FF4400 - FF44FF Hard disk ATA/IDE FF4500 - FF45FF free FF4600 - FF46FF free FF4700 - FF47FF free"
- note removed: "FF4000 - FF40FF UART0 FF4100 - FF41FF UART1 FF4200 - FF42FF UART2 FF4300 - FF43FF UART3 FF4400 - FF44FF Hard disk ATA/IDE FF4500 - FF45FF MemSlots FF4600 - FF46FF free FF4700 - FF47FF free"
Changed lines of the file:
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@@
 		)
 	)
-	(text "FF4000 - FF40FF   UART0\nFF4100 - FF41FF   UART1\nFF4200 - FF42FF   UART2\nFF4300 - FF43FF   UART3\nFF4400 - FF44FF   Hard disk ATA/IDE \nFF4500 - FF45FF   MemSlots\nFF4600 - FF46FF   free  \nFF4700 - FF47FF   free  "
+	(text "FF4000 - FF40FF   UART0\nFF4100 - FF41FF   UART1\nFF4200 - FF42FF   UART2\nFF4300 - FF43FF   UART3\nFF4400 - FF44FF   Hard disk ATA/IDE \nFF4500 - FF45FF   free\nFF4600 - FF46FF   free  \nFF4700 - FF47FF   free  "
 		(exclude_from_sim no)
 		(at 351.028 36.576 0)
@@
 	)
 	(label "{slash}AS"
-		(at 344.17 78.74 180)
+		(at 379.73 74.93 180)
 		(effects
 			(font
@@
 	)
 	(label "A11"
-		(at 379.73 74.93 180)
+		(at 344.17 78.74 180)
 		(effects
 			(font
