File: schematics/Orion68/ide_driver.kicad_sch (KiCad schematic)
At the start: 10 parts, among them J10 IDE-40W, J6 Euro96pin, U24 RP2350B, U27 74HC245, U37 GAL22V10, U38 74HC245, U39 74HC245, U40 74HC245

Commit message: 2026-09-27: implemented and tested Orionide board
Parts:
- removed U37: GAL22V10, Package_DIP:DIP-24_W7.62mm_Socket, symbol plds:GAL22V10
- added J37: Conn_02x02_Counter_Clockwise, symbol Connector_Generic:Conn_02x02_Counter_Clockwise
- added R55: 2k2, symbol Device:R
- added U19, U45: 74LS139, symbol 74xx:74LS139
- added U41: ~, symbol pdSilva:74HC4078
- added U42: 74HC138, symbol 74xx:74HC138
Connections:
- net +5V: now also U41.14 (VCC), U42.16 (VCC)
- net 5V: now also R55.2, U19.16 (VCC)
- net A10: now also U42.3 (A2)
- net A11: now also U41.5 (I4)
- net A12: now also U41.2 (I1)
- net A13: now also U41.3 (I2)
- net A14: now also U42.6 (E2)
- net A15: now also U41.4 (I3)
- net A8: now also U42.1 (A0)
- net A9: now also U42.2 (A1)
- net GND: now also U45.13 (A1); no longer J10.19 (Pin_19), J10.2 (Pin_2), J10.22 (Pin_22), J10.24 (Pin_24), J10.26 (Pin_26), J10.28 (Pin_28), J10.30 (Pin_30), J10.40 (Pin_40)
- net /AS: now also U42.4 (~{E0})
- net /CS_IDE_ATA: now also J37.3 (Pin_3), J37.4 (Pin_4), U42.11 (~{Y4}), U45.15 (E)
- net /IO_CS: now also U41.11 (I7)
- net /IO_CS1: now also U41.12 (I8)
- net /LDS: now also U45.3 (A1)
- net /RD: now also U45.11 (O1)
- net /UDS: now also U45.2 (A0)
- net /WR: now also U45.12 (O0)
- net /memwr: now also U45.14 (A0)
- net at J10.38 (Pin_38): now also R55.1
- new net: J10.19 (Pin_19), J10.2 (Pin_2), J10.22 (Pin_22), J10.24 (Pin_24), J10.26 (Pin_26), J10.28 (Pin_28), J10.30 (Pin_30), J10.40 (Pin_40)
- new net: U41.1 (O1), U42.5 (~{E1})
- new net GNDREF: U19.8 (GND), U41.10 (I6), U41.7 (VCC), U41.9 (I5), U42.8 (GND)
- new net /CSDATA: U45.4 (O0)
- new net /CSIDE: U42.15 (~{Y0}), U45.1 (E)
- new net /CSTASKFILE: U45.5 (O1)
- no-connect marks 7 -> 10
Other:
- note added: "NÃO IMPLEMENTADO"
- moved on the sheet: J10, J6, R17, R18

Commit message: 2026-09-29: updating
Connections:
- net /CS_DATA is gone; now on net /CSDATA: U40.17 (B1)
- net /CS_TASKFILE is gone; now on net /CSTASKFILE: U40.16 (B2)
- net /DS is gone; now on net /CSIDE: U40.15 (B3)
- net GND: now also J10.19 (Pin_19), J10.2 (Pin_2), J10.22 (Pin_22), J10.24 (Pin_24), J10.26 (Pin_26), J10.28 (Pin_28), J10.30 (Pin_30), J10.40 (Pin_40)
- net /CSIDE: now also U27.19 (CE), U38.19 (CE)
- net /CS_IDE: no longer U27.19 (CE), U38.19 (CE)
- net /PicoDS renamed /PicoCSIDE
Other:
- note added: "FF4000 - FF40FF picoIDE FF4100 - FF41FF free FF4200 - FF42FF free FF4300 - FF43FF free FF4400 - FF44FF Hard disk ATA/IDE FF4500 - FF45FF free FF4600 - FF46FF free FF4700 - FF47FF free"
- note added: "IDE1 = picoide IDE_REG_DATA = 0, 0xFF4000 IDE_REG_ERROR_FEATURES = 1, 0xFF4000 (1 * 2)+1 = 0xFF4003 IDE_REG_SECTOR_COUNT = 2, 0xFF4000 (2 * 2)+1 = 0xFF4005 IDE_REG_LBA_LOW = 3, 0xFF4000 (3 * 2)+1 = 0xFF4007 IDE_REG_LBA_MID = 4, 0xFF4000 (4 * 2)+1 = 0xFF4009 IDE_REG_LBA_HIGH = 5, 0xFF4000 (5 * 2)+1 = 0xFF400B IDE_REG_DEVICE_HEAD = 6, 0xFF4000 (6 * 2)+1 = 0xFF400D IDE_REG_STATUS_CMD = 7, 0xFF4000 (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"
- note removed: "IDE1 = picoide IDE_REG_DATA = 0, 0xFE0000 IDE_REG_ERROR_FEATURES = 1, 0xFE0000 (1 * 2)+1 = 0xFE0003 IDE_REG_SECTOR_COUNT = 2, 0xFE0000 (2 * 2)+1 = 0xFE0005 IDE_REG_LBA_LOW = 3, 0xFE0000 (3 * 2)+1 = 0xFE0007 IDE_REG_LBA_MID = 4, 0xFE0000 (4 * 2)+1 = 0xFE0009 IDE_REG_LBA_HIGH = 5, 0xFE0000 (5 * 2)+1 = 0xFE000B IDE_REG_DEVICE_HEAD = 6, 0xFE0000 (6 * 2)+1 = 0xFE000D IDE_REG_STATUS_CMD = 7, 0xFE0000 (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"
- moved on the sheet: J10, J37, J6, R17, R18, R55, U19C

Commit message: 2026-10-03: CHANGED FROM PIGBACK BOARD to 74hc138 + 74hc4078
Parts:
- removed J6: Euro96pin, ConnPdSilva:conn_euro96, symbol ConnPdSilva:ConnEuro96
- added J39: Euro96pin, ConnPdSilva:conn_euro96, symbol ConnPdSilva:ConnEuro96
Connections:
- net +12V: now also J39.95
- net +5V: now also J39.1, J39.33, J39.65
- net -5V: now also J39.94
- net A1: now also J39.19
- net A10: now also J39.28
- net A11: now also J39.29
- net A12: now also J39.30
- net A13: now also J39.31
- net A14: now also J39.91
- net A15: now also J39.90
- net A16: now also J39.89
- net A17: now also J39.88
- net A18: now also J39.87
- net A19: now also J39.86
- net A2: now also J39.20
- net A20: now also J39.81
- net A21: now also J39.80
- net A22: now also J39.79
- net A23: now also J39.78
- net A3: now also J39.21
- net A4: now also J39.22
- net A5: now also J39.23
- net A6: now also J39.24
- net A7: now also J39.25
- net A8: now also J39.26
- net A9: now also J39.27
- net AMARELO: now also J39.61
- net D0: now also J39.2
- net D1: now also J39.3
- net D10: now also J39.12
- net D11: now also J39.13
- net D12: now also J39.14
- net D13: now also J39.15
- net D14: now also J39.16
- net D15: now also J39.17
- net D2: now also J39.4
- net D3: now also J39.5
- net D4: now also J39.6
- net D5: now also J39.7
- net D6: now also J39.8
- net D7: now also J39.9
- net D8: now also J39.10
- net D9: now also J39.11
- net GND: now also J39.32, J39.64, J39.96
- net IRQ1: now also J39.93
- net IRQ3: now also J39.76
- net IRQ4: now also J39.77
- net IRQ5: now also J39.83
- net IRQ7: now also J39.68
- net LILAS: now also J39.59
- net MARRON: now also J39.60
- net PRETO: now also J39.57
- net RESET: now also J39.67
- net SD_CS: now also U24.47 (ADC-GP41); no longer U24.49 (ADC-GP43)
- net SD_RX(MISO): now also U24.46 (ADC-GP40); no longer U24.48 (ADC-GP42)
- net SD_SCK: now also U24.48 (ADC-GP42); no longer U24.46 (ADC-GP40)
- net SD_TX(MOSI): now also U24.49 (ADC-GP43); no longer U24.47 (ADC-GP41)
- net VERDE: now also J39.62
- net VERMELHO: now also J39.58
- net /AS: now also J39.69
- net /IO_CS: now also J39.84
- net /IO_CS1: now also J39.82
- net /LDS: now also J39.70
- net /MEM_CS: now also J39.85
- net /RESET: now also J39.66
- net /UDS: now also J39.71
- net /iord: now also J39.72
- net /iowr: now also J39.75
- net /memrd: now also J39.73
- net /memwr: now also J39.74
- net /CSIDE renamed /CS_PICOIDE
- net /CS_PICOIDE: now also J39.55
- net /DTACK_IDE renamed /DTACK_PICOIDE
- net /DTACK_PICOIDE: now also J39.54
- new net LARANJA: J39.56
- new net LILAS1: J39.63
Other:
- note removed: "LILAS"
