File: schematics/Orion68/orion68io.kicad_sch (KiCad schematic)
At the start: 45 parts, among them IC4 XR68C681CJTR-F, J1 LevelConverter, J200 Euro96pin, J22 Kbd_usb, J23 Conn_01x06, J26 DuartB, J28 DuartA, Q4 3.6864MHz, U200 GAL16V8, U25 SN74LVC245APW, U26 SN74LVC245APW, U30 LM2937xT, U33 68681, U36 UART2

Commit message: 2026-09-15: added picoIDE
Parts:
- added U16: 74HC138, symbol 74xx:74HC138
- added U21: 74HC4078, Package_DIP:DIP-14_W7.62mm, symbol pdSilva:74HC4078
- added U22: 74LS08, symbol 74xx:74LS08
Connections:
- net /CS_MULTIO_C is gone; now on net /CS_MIO: U26.7 (A6)
- net /DT_DUART is gone; now on net PRETO: U33.9 (DTACK)
- net +5V: now also U16.16 (VCC), U21.14 (VCC), U22.14 (VCC)
- net A08: now also U16.1 (A0)
- net A09: now also U16.2 (A1)
- net A10: now also U16.3 (A2)
- net A11: now also U21.2 (I1)
- net A12: now also U22.1
- net A13: now also U21.3 (I2)
- net A14: now also U21.4 (I3)
- net A15: now also U22.2
- net GND: now also U16.8 (GND), U21.11 (I7), U21.12 (I8), U21.7 (VCC), U22.7 (GND)
- net /AS: now also U21.5 (I4)
- net /CS_DUART: now also U16.15 (~{Y0})
- net /CS_MIO: now also U16.14 (~{Y1})
- net /IO_CS: now also U21.9 (I5)
- net /IO_CS1: now also U21.10 (I6)
- net /CS_RTC: no longer names the net of U200.17 (I03)
- new net: U16.6 (E2), U22.3
- new net: U16.4 (~{E0}), U16.5 (~{E1}), U21.1 (O1)
Other:
- moved on the sheet: U200

Commit message: 2026-10-03: CHANGED FROM PIGBACK BOARD to 74hc138 + 74hc4078
Parts:
- removed D_S500: LED, Diode_THT:D_T-1_P5.08mm_Horizontal, symbol Device:LED
- removed IC4: XR68C681CJTR-F, Package_LCC:PLCC-44_THT-Socket, symbol rosco_m68k-rescue:XR68C681CJTR-F-XR68C681
- removed J_S500: IDE, Connector_PinHeader_2.54mm:PinHeader_2x20_P2.54mm_Horizontal, symbol Connector_Generic:Conn_02x20_Odd_Even
- removed LED1: GREEN, rosco_m68k:LED5MM, symbol rosco_m68k-eagle-import:LED5MM
- removed LED2: RED, rosco_m68k:LED5MM, symbol rosco_m68k-eagle-import:LED5MM
- removed R56, R57: 1K, Resistor_SMD:R_0603_1608Metric, symbol rosco_m68k-eagle-import:R-EU_0207_10
- removed R_S500: 1k, Resistor_THT:R_Axial_DIN0204_L3.6mm_D1.6mm_P5.08mm_Horizontal, symbol Device:R
- removed U200: GAL16V8, Package_DIP:DIP-20_W7.62mm, symbol Logic_Programmable:GAL16V8
- added U43: 74HC4078, Package_DIP:DIP-14_W7.62mm, symbol pdSilva:74HC4078
- added U44: 74HC138, symbol 74xx:74HC138
- J23: value Conn_01x06 -> RTC
Connections:
- net /CS_DUART is gone; now on net LARANJA: U16.15 (~{Y0}), U33.35 (CS)
- net /CS_MULTIO is gone; now on net AMARELO: U25.19 (~{OE}), U26.13 (B6)
- net /DTACK_MIO is gone; now on net MARRON: U_S200.19 (GP14)
- net /DTACK_PVGA is gone; now on net LILAS: J200.59
- net +5V: now also U43.14 (VCC), U44.16 (VCC)
- net A08: now also U44.1 (A0)
- net A09: now also U44.2 (A1)
- net A11: now also U43.2 (I1)
- net A12: now also U44.3 (A2)
- net A13: now also U43.3 (I2)
- net A14: now also U43.4 (I3)
- net A15: now also U44.6 (E2)
- net AMARELO: now also U16.14 (~{Y1}), U44.10 (~{Y5})
- net CS_SDCARD: no longer U_S200.29 (GP22)
- net GND: now also U43.11 (I7), U43.12 (I8), U43.7 (VCC), U44.8 (GND)
- net LILAS: no longer J200.63
- net PRETO: no longer U33.9 (DTACK)
- net SPI1_MISO: no longer U_S200.34 (GP28)
- net SPI1_MOSI: no longer U_S200.32 (GP27)
- net SPI1_SCK: no longer U_S200.31 (GP26)
- net /AS: now also U43.5 (I4)
- net /CS_MIO: no longer U16.14 (~{Y1})
- net /IO_CS: now also U43.9 (I5)
- net /IO_CS1: now also U43.10 (I6)
- net /DTACK_PICOIDE: now reaches J200.54
- net /CS_PICOIDE: now reaches J200.55
- net LARANJA: now reaches J200.56
- net LARANJA: now also U44.11 (~{Y4})
- net SPICLK: no longer names the net of J23.2 (Pin_2)
- net SPICS: no longer names the net of J23.1 (Pin_1)
- net SPIMISO: no longer names the net of J23.4 (Pin_4)
- net SPIMOSI: no longer names the net of J23.3 (Pin_3)
- new net: U43.1 (O1), U44.4 (~{E0}), U44.5 (~{E1})
- new net LILAS1: J200.63
- new net SCL: U_S200.32 (GP27)
- new net SDA: U_S200.31 (GP26)
- new net /DTACK_68681: U33.9 (DTACK)
Other:
- note added: "FF9000->DUART -Uart1 FF9100->Super MultiIO"
- note removed: "CS"
- note removed: "LILAS"
- note removed: "MISO"
- note removed: "MOSI"
- note removed: "SCK"
- note removed: "Setor S100A"
- moved on the sheet: J23
